File: ATtiny LED badge/ATtiny LED badge.brd (EAGLE design)
At the start: 50.8 x 50.8 mm, 29 parts

Commit message: Inseriti le giunzioni mancanti nello schema
Connections:
- removed net N$7: LED14.K, LED18.K, LED3.K, LED7.K
- removed net N$8: LED11.K, LED15.K, LED19.K, LED4.K
- net N$2: now also LED11.K, LED15.K, LED19.K, LED4.K
- net N$3: now also LED14.K, LED18.K, LED3.K, LED7.K
Routing:
- net N$8: track 27.4 -> 0.00 mm
- net N$2: track 29.5 -> 56.9 mm
- net N$7: track 23.0 -> 0.00 mm
- net N$3: track 35.1 -> 58.1 mm
Changed lines of the file:
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@@
 <wire x1="21.5" y1="19" x2="21.59" y2="19.05" width="0.254" layer="16"/>
 <wire x1="17" y1="19" x2="16.51" y2="19.05" width="0.254" layer="16"/>
+<contactref element="LED19" pad="K"/>
+<contactref element="LED4" pad="K"/>
+<contactref element="LED11" pad="K"/>
+<contactref element="LED15" pad="K"/>
+<wire x1="29.5" y1="8.5" x2="29.5" y2="4" width="0.254" layer="1"/>
+<wire x1="29.5" y1="4" x2="29.21" y2="3.81" width="0.254" layer="1"/>
+<wire x1="29.5" y1="8.5" x2="29.21" y2="8.89" width="0.254" layer="1"/>
+<wire x1="29.5" y1="9" x2="29.5" y2="13.5" width="0.254" layer="1"/>
+<wire x1="29.5" y1="13.5" x2="29.21" y2="13.97" width="0.254" layer="1"/>
+<wire x1="29.5" y1="9" x2="29.21" y2="8.89" width="0.254" layer="1"/>
+<wire x1="34" y1="20.5" x2="34" y2="24" width="0.254" layer="16"/>
+<wire x1="33" y1="19.5" x2="34" y2="20.5" width="0.254" layer="16"/>
+<wire x1="33" y1="12.5" x2="33" y2="19.5" width="0.254" layer="16"/>
+<wire x1="30.5" y1="12.5" x2="33" y2="12.5" width="0.254" layer="16"/>
+<wire x1="29.5" y1="13.5" x2="30.5" y2="12.5" width="0.254" layer="16"/>
+<wire x1="34" y1="24" x2="34.29" y2="24.13" width="0.254" layer="16"/>
+<wire x1="29.5" y1="13.5" x2="29.21" y2="13.97" width="0.254" layer="16"/>
+<wire x1="33" y1="19.5" x2="31.75" y2="19.05" width="0" layer="19" extent="16-16"/>
 </signal>
 <signal name="N$3">
@@
 <wire x1="25.5" y1="15" x2="30.5" y2="15" width="0.254" layer="16"/>
 <wire x1="31.5" y1="14" x2="31.75" y2="13.97" width="0.254" layer="16"/>
+<contactref element="LED18" pad="K"/>
+<contactref element="LED3" pad="K"/>
+<contactref element="LED7" pad="K"/>
+<contactref element="LED14" pad="K"/>
+<wire x1="24" y1="8.5" x2="24" y2="4" width="0.254" layer="1"/>
+<wire x1="24" y1="4" x2="24.13" y2="3.81" width="0.254" layer="1"/>
+<wire x1="24" y1="8.5" x2="24.13" y2="8.89" width="0.254" layer="1"/>
+<wire x1="29.5" y1="24" x2="29.5" y2="19.5" width="0.254" layer="1"/>
+<wire x1="29.5" y1="19.5" x2="29.21" y2="19.05" width="0.254" layer="1"/>
+<wire x1="29.5" y1="24" x2="29.21" y2="24.13" width="0.254" layer="1"/>
+<wire x1="28" y1="12.5" x2="24.5" y2="9" width="0.254" layer="1"/>
+<wire x1="28" y1="18" x2="28" y2="12.5" width="0.254" layer="1"/>
+<wire x1="29" y1="19" x2="28" y2="18" width="0.254" layer="1"/>
+<wire x1="24.5" y1="9" x2="24.13" y2="8.89" width="0.254" layer="1"/>
+<wire x1="29" y1="19" x2="29.21" y2="19.05" width="0.254" layer="1"/>
+<wire x1="26.67" y1="13.97" x2="28" y2="12.5" width="0" layer="19" extent="1-1"/>
 </signal>
 <signal name="N$4">
@@
 <wire x1="19" y1="14" x2="19.05" y2="13.97" width="0.254" layer="1"/>
 </signal>
-<signal name="N$7">
-<contactref element="LED18" pad="K"/>
-<contactref element="LED3" pad="K"/>
-<contactref element="LED7" pad="K"/>
-<contactref element="LED14" pad="K"/>
-<wire x1="24" y1="8.5" x2="24" y2="4" width="0.254" layer="1"/>
-<wire x1="24" y1="4" x2="24.13" y2="3.81" width="0.254" layer="1"/>
-<wire x1="24" y1="8.5" x2="24.13" y2="8.89" width="0.254" layer="1"/>
-<wire x1="29.5" y1="24" x2="29.5" y2="19.5" width="0.254" layer="1"/>
-<wire x1="29.5" y1="19.5" x2="29.21" y2="19.05" width="0.254" layer="1"/>
-<wire x1="29.5" y1="24" x2="29.21" y2="24.13" width="0.254" layer="1"/>
-<wire x1="28" y1="12.5" x2="24.5" y2="9" width="0.254" layer="1"/>
-<wire x1="28" y1="18" x2="28" y2="12.5" width="0.254" layer="1"/>
-<wire x1="29" y1="19" x2="28" y2="18" width="0.254" layer="1"/>
-<wire x1="24.5" y1="9" x2="24.13" y2="8.89" width="0.254" layer="1"/>
-<wire x1="29" y1="19" x2="29.21" y2="19.05" width="0.254" layer="1"/>
-</signal>
-<signal name="N$8">
-<contactref element="LED19" pad="K"/>
-<contactref element="LED4" pad="K"/>
-<contactref element="LED11" pad="K"/>
-<contactref element="LED15" pad="K"/>
-<wire x1="29.5" y1="8.5" x2="29.5" y2="4" width="0.254" layer="1"/>
-<wire x1="29.5" y1="4" x2="29.21" y2="3.81" width="0.254" layer="1"/>
-<wire x1="29.5" y1="8.5" x2="29.21" y2="8.89" width="0.254" layer="1"/>
-<wire x1="29.5" y1="9" x2="29.5" y2="13.5" width="0.254" layer="1"/>
-<wire x1="29.5" y1="13.5" x2="29.21" y2="13.97" width="0.254" layer="1"/>
-<wire x1="29.5" y1="9" x2="29.21" y2="8.89" width="0.254" layer="1"/>
-<wire x1="34" y1="20.5" x2="34" y2="24" width="0.254" layer="16"/>
-<wire x1="33" y1="19.5" x2="34" y2="20.5" width="0.254" layer="16"/>
-<wire x1="33" y1="12.5" x2="33" y2="19.5" width="0.254" layer="16"/>
-<wire x1="30.5" y1="12.5" x2="33" y2="12.5" width="0.254" layer="16"/>
-<wire x1="29.5" y1="13.5" x2="30.5" y2="12.5" width="0.254" layer="16"/>
-<wire x1="34" y1="24" x2="34.29" y2="24.13" width="0.254" layer="16"/>
-<wire x1="29.5" y1="13.5" x2="29.21" y2="13.97" width="0.254" layer="16"/>
-</signal>
 <signal name="N$6">
