File: ATtiny LED badge/ATtiny LED badge.brd (EAGLE design)
At the start: 50.8 x 50.8 mm, 29 parts

Commit message: routed PCBs
Parts:
- moved R5 18.5 mm to (15.9, 33.0), turned to 270 degrees
- moved IC1 14.0 mm to (25.4, 33.0), flipped to the bottom
- moved R4 13.7 mm to (12.7, 33.0), turned to 270 degrees
- moved R3 9.09 mm to (9.53, 33.0), turned to 270 degrees
- moved R1 8.98 mm to (44.5, 25.4), turned to 180 degrees
- moved R2 5.24 mm to (6.35, 33.0), turned to 270 degrees
- moved JP1 2.54 mm to (44.5, 30.5)
- moved LED1 0.64 mm to (17.8, 24.8), turned to 315 degrees
- moved LED2 0.64 mm to (22.9, 24.8), turned to 315 degrees
- moved LED3 0.64 mm to (27.9, 24.8), turned to 315 degrees
- moved LED4 0.64 mm to (33.0, 24.8), turned to 315 degrees
- moved LED17 0.64 mm to (17.8, 4.45), turned to 315 degrees
- moved LED18 0.64 mm to (22.9, 4.45), turned to 315 degrees
- moved LED19 0.64 mm to (27.9, 4.45), turned to 315 degrees
- moved LED20 0.64 mm to (33.0, 4.45), turned to 315 degrees
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Routing:
- net MOSI: track 49.5 -> 31.8 mm
- net SCK: track 55.5 -> 38.1 mm
- net PB4: track 23.2 -> 7.44 mm
- net MISO: track 55.4 -> 43.8 mm
- net N$5: track 51.7 -> 42.7 mm
- net RST: track 28.4 -> 20.2 mm, vias 1 -> 0
- net PB3: track 18.0 -> 11.1 mm, vias 1 -> 0
- net GND: track 34.4 -> 27.7 mm, vias 0 -> 1
- net N$1: track 49.6 -> 46.7 mm
- net N$4: track 53.5 -> 51.4 mm
- net N$3: track 55.6 -> 53.8 mm
- net N$2: track 52.4 -> 51.2 mm
- net N$6: track 28.9 -> 27.7 mm
- net VCC: track 58.4 -> 58.7 mm, vias 1 -> 0

Commit message: renderings + gerbers
Routing:
- net VCC: track 58.7 -> 58.0 mm
Changed lines of the file:
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@@
 <layer number="28" name="bValues" color="7" fill="1" visible="yes" active="yes"/>
 <layer number="29" name="tStop" color="7" fill="3" visible="no" active="yes"/>
-<layer number="30" name="bStop" color="7" fill="6" visible="no" active="yes"/>
+<layer number="30" name="bStop" color="7" fill="6" visible="yes" active="yes"/>
 <layer number="31" name="tCream" color="7" fill="4" visible="no" active="yes"/>
 <layer number="32" name="bCream" color="7" fill="5" visible="no" active="yes"/>
@@
 <rectangle x1="16.51" y1="44.45" x2="34.29" y2="48.26" layer="16"/>
 <circle x="15.24" y="26.67" radius="0.635" width="0" layer="21"/>
+<rectangle x1="16.51" y1="44.45" x2="34.29" y2="48.26" layer="30"/>
 </plain>
 <attributes>
@@
 <wire x1="21.59" y1="34.915" x2="21.996" y2="34.915" width="0.3" layer="16"/>
 <wire x1="21.996" y1="34.915" x2="24.12" y2="34.915" width="0.3" layer="16"/>
-<wire x1="24.12" y1="34.915" x2="24.765" y2="35.56" width="0.3" layer="16"/>
-<wire x1="24.765" y1="35.56" x2="35.56" y2="35.56" width="0.3" layer="16"/>
+<wire x1="24.12" y1="34.915" x2="26.67" y2="35.56" width="0.3" layer="16"/>
+<wire x1="26.67" y1="35.56" x2="35.56" y2="35.56" width="0.3" layer="16"/>
 <via x="35.56" y="35.56" extent="1-16" drill="0.7"/>
 <wire x1="35.56" y1="35.56" x2="41.91" y2="29.21" width="0.3" layer="1"/>
@@
 <contactref element="JP1" pad="2"/>
 <contactref element="JP2" pad="2"/>
-<wire x1="28.804" y1="31.115" x2="26.035" y2="31.115" width="0.3" layer="16"/>
-<wire x1="26.035" y1="31.115" x2="25.4" y2="30.48" width="0.3" layer="16"/>
-<wire x1="25.4" y1="30.48" x2="10.795" y2="30.48" width="0.3" layer="16"/>
+<wire x1="28.804" y1="31.115" x2="26.67" y2="31.115" width="0.3" layer="16"/>
+<wire x1="26.67" y1="31.115" x2="24.13" y2="30.48" width="0.3" layer="16"/>
+<wire x1="24.13" y1="30.48" x2="10.795" y2="30.48" width="0.3" layer="16"/>
 <wire x1="10.795" y1="30.48" x2="5.08" y2="36.195" width="0.3" layer="16"/>
 <wire x1="5.08" y1="36.195" x2="5.08" y2="37.465" width="0.3" layer="16"/>
-<wire x1="5.08" y1="37.465" x2="7.62" y2="40.005" width="0.3" layer="16"/>
-<wire x1="7.62" y1="40.005" x2="12.7" y2="40.005" width="0.3" layer="16"/>
+<wire x1="5.08" y1="37.465" x2="6.35" y2="38.735" width="0.3" layer="16"/>
+<wire x1="28.804" y1="31.115" x2="38.1" y2="31.115" width="0.3" layer="16"/>
+<wire x1="38.1" y1="31.115" x2="41.275" y2="27.94" width="0.3" layer="16"/>
+<wire x1="41.275" y1="27.94" x2="45.72" y2="27.94" width="0.3" layer="16"/>
+<wire x1="45.72" y1="27.94" x2="46.99" y2="29.21" width="0.3" layer="16"/>
+<wire x1="6.35" y1="38.735" x2="11.43" y2="38.735" width="0.3" layer="16"/>
+<wire x1="11.43" y1="38.735" x2="12.7" y2="40.005" width="0.3" layer="16"/>
 <wire x1="12.7" y1="40.005" x2="12.7" y2="41.91" width="0.3" layer="16"/>
-<wire x1="46.99" y1="29.21" x2="45.72" y2="27.94" width="0.3" layer="16"/>
-<wire x1="45.72" y1="27.94" x2="31.115" y2="27.94" width="0.3" layer="16"/>
-<wire x1="31.115" y1="27.94" x2="28.804" y2="30.251" width="0.3" layer="16"/>
-<wire x1="28.804" y1="30.251" x2="28.804" y2="31.115" width="0.3" layer="16"/>
 </signal>
 <signal name="MISO">
@@
 <wire x1="16.51" y1="38.1" x2="20.32" y2="34.29" width="0.3" layer="16"/>
 <wire x1="20.32" y1="34.29" x2="24.13" y2="34.29" width="0.3" layer="16"/>
-<wire x1="24.13" y1="34.29" x2="24.765" y2="33.655" width="0.3" layer="16"/>
-<wire x1="24.765" y1="33.655" x2="28.804" y2="33.655" width="0.3" layer="16"/>
+<wire x1="24.13" y1="34.29" x2="26.67" y2="33.655" width="0.3" layer="16"/>
+<wire x1="26.67" y1="33.655" x2="28.804" y2="33.655" width="0.3" layer="16"/>
 <wire x1="28.804" y1="33.655" x2="45.085" y2="33.655" width="0.3" layer="16"/>
 <wire x1="45.085" y1="33.655" x2="46.99" y2="31.75" width="0.3" layer="16"/>
@@
 <wire x1="9.525" y1="36.83" x2="14.605" y2="31.75" width="0.3" layer="16"/>
 <wire x1="14.605" y1="31.75" x2="24.13" y2="31.75" width="0.3" layer="16"/>
-<wire x1="24.13" y1="31.75" x2="24.765" y2="32.385" width="0.3" layer="16"/>
-<wire x1="24.765" y1="32.385" x2="28.804" y2="32.385" width="0.3" layer="16"/>
-<wire x1="28.804" y1="32.385" x2="34.29" y2="32.385" width="0.3" layer="16"/>
-<wire x1="34.29" y1="32.385" x2="34.925" y2="33.02" width="0.3" layer="16"/>
-<wire x1="34.925" y1="33.02" x2="43.18" y2="33.02" width="0.3" layer="16"/>
+<wire x1="24.13" y1="31.75" x2="26.67" y2="32.385" width="0.3" layer="16"/>
+<wire x1="26.67" y1="32.385" x2="28.804" y2="32.385" width="0.3" layer="16"/>
+<wire x1="28.804" y1="32.385" x2="40.64" y2="32.385" width="0.3" layer="16"/>
+<wire x1="40.64" y1="32.385" x2="41.275" y2="33.02" width="0.3" layer="16"/>
+<wire x1="41.275" y1="33.02" x2="43.18" y2="33.02" width="0.3" layer="16"/>
 <wire x1="43.18" y1="33.02" x2="44.45" y2="31.75" width="0.3" layer="16"/>
 </signal>
@@
 <contactref element="JP1" pad="5"/>
 <contactref element="IC1" pad="1"/>
-<wire x1="21.996" y1="31.115" x2="24.765" y2="31.115" width="0.3" layer="16"/>
-<wire x1="24.765" y1="31.115" x2="25.4" y2="31.75" width="0.3" layer="16"/>
-<wire x1="25.4" y1="31.75" x2="41.91" y2="31.75" width="0.3" layer="16"/>
+<wire x1="21.996" y1="31.115" x2="24.13" y2="31.115" width="0.3" layer="16"/>
+<wire x1="24.13" y1="31.115" x2="26.67" y2="31.75" width="0.3" layer="16"/>
+<wire x1="26.67" y1="31.75" x2="41.91" y2="31.75" width="0.3" layer="16"/>
 </signal>
 <signal name="MOSI">
