File: ATtiny LED badge/ATtiny LED badge.brd (EAGLE design)
At the start: 50.8 x 50.8 mm, 29 parts

Commit message: updated to ATtiny13
Parts:
- IC1: value (none) -> TINY13-20SSU; device atmel:8S2 -> atmel:8S1
Routing:
- net RST: track 20.0 -> 19.2 mm
- net PB4: track 7.44 -> 8.19 mm
- net PB3: track 11.1 -> 11.9 mm
- net MOSI: track 31.8 -> 32.5 mm
Changed lines of the file:
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@@
 <?xml version="1.0" encoding="utf-8"?>
 <!DOCTYPE eagle SYSTEM "eagle.dtd">
-<eagle version="7.6.0">
+<eagle version="8.4.3">
 <drawing>
 <settings>
 <setting alwaysvectorfont="no"/>
+<setting keepoldvectorfont="yes"/>
 <setting verticaltext="up"/>
 </settings>
@@
 <layers>
 <layer number="1" name="Top" color="4" fill="1" visible="yes" active="yes"/>
+<layer number="2" name="Route2" color="1" fill="3" visible="no" active="no"/>
+<layer number="3" name="Route3" color="4" fill="3" visible="no" active="no"/>
+<layer number="4" name="Route4" color="1" fill="4" visible="no" active="no"/>
+<layer number="5" name="Route5" color="4" fill="4" visible="no" active="no"/>
+<layer number="6" name="Route6" color="1" fill="8" visible="no" active="no"/>
+<layer number="7" name="Route7" color="4" fill="8" visible="no" active="no"/>
+<layer number="8" name="Route8" color="1" fill="2" visible="no" active="no"/>
+<layer number="9" name="Route9" color="4" fill="2" visible="no" active="no"/>
+<layer number="10" name="Route10" color="1" fill="7" visible="no" active="no"/>
+<layer number="11" name="Route11" color="4" fill="7" visible="no" active="no"/>
+<layer number="12" name="Route12" color="1" fill="5" visible="no" active="no"/>
+<layer number="13" name="Route13" color="4" fill="5" visible="no" active="no"/>
+<layer number="14" name="Route14" color="1" fill="6" visible="no" active="no"/>
+<layer number="15" name="Route15" color="4" fill="6" visible="no" active="no"/>
 <layer number="16" name="Bottom" color="1" fill="1" visible="yes" active="yes"/>
 <layer number="17" name="Pads" color="2" fill="1" visible="yes" active="yes"/>
@@
 <param name="dpMaxLengthDifference" value="10mm"/>
 <param name="dpGapFactor" value="2.5"/>
-<param name="checkGrid" value="0"/>
 <param name="checkAngle" value="0"/>
 <param name="checkFont" value="1"/>
 <param name="checkRestrict" value="1"/>
+<param name="checkStop" value="0"/>
 <param name="useDiameter" value="13"/>
 <param name="maxErrors" value="50"/>
@@
 <elements>
 <element name="BATTERY_1" library="Itead_BP_110825.lbr" package="BATTERY_1236_C" value="" x="41.91" y="39.37" rot="R90"/>
-<element name="IC1" library="atmel" package="8S2" value="" x="25.4" y="33.02" rot="MR90">
-<attribute name="OC_FARNELL" value="9171568" x="25.4" y="33.02" size="1.778" layer="28" rot="MR90" display="off"/>
-<attribute name="OC_NEWARK" value="96K6522" x="25.4" y="33.02" size="1.778" layer="28" rot="MR90" display="off"/>
-<attribute name="MPN" value="ATTINY13-20SU" x="25.4" y="33.02" size="1.778" layer="28" rot="MR90" display="off"/>
+<element name="IC1" library="atmel" library_urn="urn:adsk.eagle:library:105" package="8S1" package3d_urn="urn:adsk.eagle:package:4358/1" value="TINY13-20SSU" x="25.4" y="33.02" rot="MR90">
 <attribute name="MF" value="" x="25.4" y="33.02" size="1.778" layer="28" rot="MR90" display="off"/>
+<attribute name="MPN" value="ATTINY13-20SSU" x="25.4" y="33.02" size="1.778" layer="28" rot="MR90" display="off"/>
+<attribute name="OC_FARNELL" value="1455133" x="25.4" y="33.02" size="1.778" layer="28" rot="MR90" display="off"/>
+<attribute name="OC_NEWARK" value="58M3771" x="25.4" y="33.02" size="1.778" layer="28" rot="MR90" display="off"/>
 </element>
 <element name="JP1" library="pinhead" package="2X03" value="" x="44.45" y="30.48" rot="R180"/>
@@
 <contactref element="JP1" pad="6"/>
 <wire x1="21.59" y1="39.37" x2="21.59" y2="34.915" width="0.3" layer="16"/>
-<wire x1="21.59" y1="34.915" x2="21.996" y2="34.915" width="0.3" layer="16"/>
-<wire x1="21.996" y1="34.915" x2="24.12" y2="34.915" width="0.3" layer="16"/>
+<wire x1="21.59" y1="34.915" x2="22.746" y2="34.915" width="0.3" layer="16"/>
+<wire x1="22.746" y1="34.915" x2="24.12" y2="34.915" width="0.3" layer="16"/>
 <wire x1="24.12" y1="34.915" x2="26.67" y2="35.56" width="0.3" layer="16"/>
 <wire x1="26.67" y1="35.56" x2="35.56" y2="35.56" width="0.3" layer="16"/>
@@
 <contactref element="JP1" pad="2"/>
 <contactref element="JP2" pad="2"/>
-<wire x1="28.804" y1="31.115" x2="26.67" y2="31.115" width="0.3" layer="16"/>
+<wire x1="28.054" y1="31.115" x2="26.67" y2="31.115" width="0.3" layer="16"/>
 <wire x1="26.67" y1="31.115" x2="24.13" y2="30.48" width="0.3" layer="16"/>
 <wire x1="24.13" y1="30.48" x2="10.795" y2="30.48" width="0.3" layer="16"/>
@@
 <wire x1="5.08" y1="36.195" x2="5.08" y2="37.465" width="0.3" layer="16"/>
 <wire x1="5.08" y1="37.465" x2="6.35" y2="38.735" width="0.3" layer="16"/>
-<wire x1="28.804" y1="31.115" x2="38.1" y2="31.115" width="0.3" layer="16"/>
+<wire x1="28.054" y1="31.115" x2="38.1" y2="31.115" width="0.3" layer="16"/>
 <wire x1="38.1" y1="31.115" x2="41.275" y2="27.94" width="0.3" layer="16"/>
 <wire x1="41.275" y1="27.94" x2="45.72" y2="27.94" width="0.3" layer="16"/>
@@
 <wire x1="20.32" y1="34.29" x2="24.13" y2="34.29" width="0.3" layer="16"/>
 <wire x1="24.13" y1="34.29" x2="26.67" y2="33.655" width="0.3" layer="16"/>
-<wire x1="26.67" y1="33.655" x2="28.804" y2="33.655" width="0.3" layer="16"/>
-<wire x1="28.804" y1="33.655" x2="45.085" y2="33.655" width="0.3" layer="16"/>
+<wire x1="26.67" y1="33.655" x2="28.054" y2="33.655" width="0.3" layer="16"/>
+<wire x1="28.054" y1="33.655" x2="45.085" y2="33.655" width="0.3" layer="16"/>
 <wire x1="45.085" y1="33.655" x2="46.99" y2="31.75" width="0.3" layer="16"/>
 </signal>
@@
 <wire x1="14.605" y1="31.75" x2="24.13" y2="31.75" width="0.3" layer="16"/>
 <wire x1="24.13" y1="31.75" x2="26.67" y2="32.385" width="0.3" layer="16"/>
-<wire x1="26.67" y1="32.385" x2="28.804" y2="32.385" width="0.3" layer="16"/>
-<wire x1="28.804" y1="32.385" x2="40.64" y2="32.385" width="0.3" layer="16"/>
+<wire x1="26.67" y1="32.385" x2="28.054" y2="32.385" width="0.3" layer="16"/>
+<wire x1="28.054" y1="32.385" x2="40.64" y2="32.385" width="0.3" layer="16"/>
 <wire x1="40.64" y1="32.385" x2="41.275" y2="33.02" width="0.3" layer="16"/>
 <wire x1="41.275" y1="33.02" x2="43.18" y2="33.02" width="0.3" layer="16"/>
@@
 <contactref element="JP1" pad="5"/>
 <contactref element="IC1" pad="1"/>
-<wire x1="21.996" y1="31.115" x2="24.13" y2="31.115" width="0.3" layer="16"/>
+<wire x1="22.746" y1="31.115" x2="24.13" y2="31.115" width="0.3" layer="16"/>
 <wire x1="24.13" y1="31.115" x2="26.67" y2="31.75" width="0.3" layer="16"/>
 <wire x1="26.67" y1="31.75" x2="41.91" y2="31.75" width="0.3" layer="16"/>
@@
 <wire x1="48.26" y1="25.4" x2="44.45" y2="29.21" width="0.3" layer="1"/>
 <wire x1="44.45" y1="29.21" x2="45.72" y2="30.48" width="0.3" layer="16"/>
-<wire x1="28.804" y1="34.925" x2="29.845" y2="34.925" width="0.3" layer="16"/>
+<wire x1="28.054" y1="34.925" x2="29.845" y2="34.925" width="0.3" layer="16"/>
 <wire x1="29.845" y1="34.925" x2="30.48" y2="34.29" width="0.3" layer="16"/>
 <wire x1="30.48" y1="34.29" x2="46.355" y2="34.29" width="0.3" layer="16"/>
@@
 <contactref element="IC1" pad="2"/>
 <contactref element="R4" pad="1"/>
-<wire x1="21.996" y1="32.375" x2="17.155" y2="32.375" width="0.3" layer="16"/>
+<wire x1="22.746" y1="32.375" x2="17.155" y2="32.375" width="0.3" layer="16"/>
 <wire x1="17.155" y1="32.375" x2="12.7" y2="36.83" width="0.3" layer="16"/>
 </signal>
@@
 <contactref element="IC1" pad="3"/>
 <contactref element="R5" pad="1"/>
-<wire x1="21.996" y1="33.645" x2="19.06" y2="33.645" width="0.3" layer="16"/>
+<wire x1="22.746" y1="33.645" x2="19.06" y2="33.645" width="0.3" layer="16"/>
 <wire x1="19.06" y1="33.645" x2="15.875" y2="36.83" width="0.3" layer="16"/>
 </signal>
@@
 </board>
 </drawing>
+<compatibility>
+<note version="8.2" severity="warning">
+Since Version 8.2, EAGLE supports online libraries. The ids
+of those online libraries will not be understood (or retained)
+with this version.
+</note>
+<note version="8.3" severity="warning">
+Since Version 8.3, EAGLE supports URNs for individual library
+assets (packages, symbols, and devices). The URNs of those assets
+will not be understood (or retained) with this version.
+</note>
+<note version="8.3" severity="warning">
+Since Version 8.3, EAGLE supports the association of 3D packages
+with devices in libraries, schematics, and board files. Those 3D
+packages will not be understood (or retained) with this version.
+</note>
+</compatibility>
 </eagle>
