File: ATtiny badge/ATtiny badge.brd (EAGLE design)
At the start: 50.8 x 50.8 mm, 4 parts, among them IC1 TINY13-20SSU

Commit message: new badges
Parts:
- added JP3: 1, pinhead:1X01
- added JP4: 2, pinhead:1X01
- added JP5: 3, pinhead:1X01
- added JP6: 4, pinhead:1X01
- added JP7: V+, pinhead:1X01
- added JP8: GND, pinhead:1X01
- added JP9: ON, pinhead:1X03
- BATTERY_1: value BATTERY_1236_C -> (none)
- IC1: value TINY13-20SSU -> (none); device atmel:8S1 -> atmel:8S2
- JP2: value (none) -> 0; device pinhead:2X07 -> pinhead:1X01
- moved JP2 3.81 mm to (6.35, 30.5), turned to 180 degrees
- moved IC1 2.84 mm to (11.4, 36.8), turned to 90 degrees
- moved JP1 1.27 mm to (44.5, 31.8)
Connections:
- new net MISO: IC1.6, JP1.1, JP3.1
- new net MOSI: IC1.5, JP1.4, JP2.1
- new net PB3: IC1.2, JP5.1
- new net PB4: IC1.3, JP6.1
- new net RST: IC1.1, JP1.5
- new net SCK: IC1.7, JP1.3, JP4.1
- net GND: now also JP1.6, JP8.1
- net N$1: now also BATTERY_1.+, JP9.1; no longer JP2.1, JP2.2
- net VCC: now also JP1.2, JP7.1, JP9.2; no longer BATTERY_1.+
Routing:
- net GND: track 0.00 -> 70.2 mm
- net VCC: track 0.00 -> 62.0 mm
- net MISO: track 0.00 -> 50.5 mm
- net MOSI: track 0.00 -> 50.1 mm
- net SCK: track 0.00 -> 43.6 mm
- net N$1: track 0.00 -> 28.9 mm
- net RST: track 0.00 -> 28.5 mm, vias 0 -> 1
- net PB4: track 0.00 -> 7.82 mm
- net PB3: track 0.00 -> 7.35 mm

Commit message: routed PCBs
Parts:
- moved IC1 20.4 mm to (31.8, 35.6), flipped to the bottom
Routing:
- net RST: track 28.5 -> 13.8 mm, vias 1 -> 0
- net PB3: track 7.35 -> 18.4 mm
- net GND: track 70.2 -> 60.7 mm
- net PB4: track 7.82 -> 14.9 mm
- net SCK: track 43.6 -> 37.6 mm
- net MISO: track 50.5 -> 46.4 mm
- net VCC: track 62.0 -> 58.0 mm
- net MOSI: track 50.1 -> 48.7 mm, vias 0 -> 1
- net N$1: track 28.9 -> 28.2 mm

Commit message: renderings + gerbers
Parts:
- JP2: value 0 -> 0
- JP3: value 1 -> 1
- JP4: value 2 -> 2
- JP5: value 3 -> 3
- JP6: value 4 -> 4
Changed lines of the file:
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@@
 <layer number="28" name="bValues" color="7" fill="1" visible="yes" active="yes"/>
 <layer number="29" name="tStop" color="7" fill="3" visible="no" active="yes"/>
-<layer number="30" name="bStop" color="7" fill="6" visible="no" active="yes"/>
+<layer number="30" name="bStop" color="7" fill="6" visible="yes" active="yes"/>
 <layer number="31" name="tCream" color="7" fill="4" visible="no" active="yes"/>
 <layer number="32" name="bCream" color="7" fill="5" visible="no" active="yes"/>
@@
 <circle x="46.99" y="35.56" radius="0.635" width="0" layer="21"/>
 <rectangle x1="16.51" y1="44.45" x2="34.29" y2="48.26" layer="16"/>
+<rectangle x1="16.51" y1="44.45" x2="34.29" y2="48.26" layer="30"/>
 </plain>
 <attributes>
@@
 </element>
 <element name="JP1" library="pinhead" package="2X03" value="" x="44.45" y="31.75" rot="R180"/>
-<element name="JP2" library="pinhead" package="1X01" value="0  " x="6.35" y="30.48" rot="R180"/>
-<element name="JP3" library="pinhead" package="1X01" value="1  " x="8.89" y="30.48" rot="R180"/>
-<element name="JP4" library="pinhead" package="1X01" value="2  " x="11.43" y="30.48" rot="R180"/>
-<element name="JP5" library="pinhead" package="1X01" value="3  " x="13.97" y="30.48" rot="R180"/>
-<element name="JP6" library="pinhead" package="1X01" value="4  " x="16.51" y="30.48" rot="R180"/>
+<element name="JP2" library="pinhead" package="1X01" value="0" x="6.35" y="30.48" rot="R180"/>
+<element name="JP3" library="pinhead" package="1X01" value="1" x="8.89" y="30.48" rot="R180"/>
+<element name="JP4" library="pinhead" package="1X01" value="2" x="11.43" y="30.48" rot="R180"/>
+<element name="JP5" library="pinhead" package="1X01" value="3" x="13.97" y="30.48" rot="R180"/>
+<element name="JP6" library="pinhead" package="1X01" value="4" x="16.51" y="30.48" rot="R180"/>
 <element name="JP7" library="pinhead" package="1X01" value="V+" x="19.05" y="30.48" rot="R180"/>
 <element name="JP8" library="pinhead" package="1X01" value="GND" x="3.81" y="30.48" rot="R180"/>
