File: Kids badge/Kids badge.brd (EAGLE design)
At the start: 50.8 x 50.8 mm, 4 parts

Commit message: ladybug
Parts:
- removed JP1: (no value), pinhead:1X03
- added J1: (no value), SparkFun-Connectors:1X03_LOCK
- moved LED1 3.70 mm to (15.9, 37.5)
- moved LED2 3.70 mm to (34.9, 37.5)
Connections:
- net N$2: now also J1.1; no longer JP1.1
- net N$3: now also J1.2; no longer JP1.2
Routing:
- net N$2: track 24.1 -> 26.2 mm
- net N$3: track 22.2 -> 20.8 mm
- net N$1: track 46.8 -> 47.7 mm
Other:
- board text added: "1.Spilla"
- board text added: "2.LED Dal lato opposto. Attenzione alla sagoma!"
- board text added: "3.Interruttore Dal lato opposto."
- board text added: "4.Porta-batteria Da questo lato. Attenzione alla sagoma!"
