File: Ladybug/Ladybug.brd (EAGLE design)
At the start: 42.3 x 50.8 mm, 8 parts

Commit message: updated to ATtiny13
Other:
- board text added: "Motore Incollalo da questo lato dopo aver saldato il connettore."
- board text added: "Porta-batteria Tutti i componenti su questo lato. Fai attenzione alla sagoma!"
- board text removed: "Motore Incollare da questo lato dopo aver saldato il connettore."
- board text removed: "Porta-batteria Tutti i componenti su questo lato. Attenzione alla sagoma!"
