File: ATtinyNode/PCB/ATtinyNode.sch (EAGLE design)
At the start: 8 parts, among them IC1 TINY13-20SU, J1 AVR_SPI_PROG_3X2NS

Commit message: ATtinyNode review
Parts:
- removed C1: (no value), rcl:C-EUC0603
- removed IC1: TINY13-20SU, atmel:TINY13-20SU
- removed JP1: (no value), adafruit:PINHD-1X1CB
- removed JP2: (no value), adafruit:PINHD-1X3
- removed R1: (no value), rcl:R-US_R0603
- added ANT: (no value), adafruit:PINHD-1X1CB
- added C: 0.1 uF, rcl:C-EUC0805
- added DIO0/PB3, MISO/PB0: JUMPER-SMT_2_NO_SILK, SparkFun-Jumpers:JUMPER-SMT_2_NO_SILK
- added IC2: ATTINY85-20SU, ATTINY85-20SU:ATTINY85-20SU
- added J2: (no value), SparkFun-Connectors:CONN_04X2
- added R: 10k, rcl:R-US_R0805
- added U$2: FABLABAQ_LOGONONE, FabLab eagle logo:FABLABAQ_LOGONONE
- added U$3: CERN_OHL_1.2, CERN_OHL_1.2:CERN_OHL_1.2
- BT1: value (none) -> CR2032
- J1: value AVR_SPI_PROG_3X2NS -> AVR_SPI_PROG_3X2PTH; device SparkFun-Connectors:AVR_SPI_PROG_3X2NS -> SparkFun-Connectors:AVR_SPI_PROG_3X2PTH
Connections:
- removed net B1: U$1.DIO2
- removed net DIO1: U$1.DIO1
- removed net DIO3: U$1.DIO3
- removed net DIO4: U$1.DIO4
- removed net DIO5: U$1.DIO5
- removed net N$20: BT1.+, JP2.1
- removed net SCK: U$1.SCK
- new net DIO0: DIO0/PB3.1, U$1.DIO0
- net ANT: now also ANT.1; no longer JP1.1
- net GND: now also C.2, IC2.GND, J2.1; no longer C1.2, IC1.GND
- net MISO: now also MISO/PB0.1
- net PB0: now also IC2.MOSI, J2.2, MISO/PB0.2; no longer IC1.PB0/PCINT0/AIN0/OC0A/MOSI
- net PB1: now also IC2.MISO, J2.4; no longer IC1.PB1/PCINT1/AIN1/OC0B/INT0/MISO
- net PB2: now also IC2.SCK, J2.6, U$1.SCK; no longer IC1.PB2/PCINT2/SCK/ADC1/T0
- net PB3: now also DIO0/PB3.2, IC2.PCINT3, J2.5; no longer IC1.PB3/PCINT3/CLKI/ADC3, U$1.DIO0
- net PB4: now also IC2.PCINT4, J2.3; no longer IC1.PB4/PCINT4/ADC2
- net RST: now also IC2.PCINT5, J2.7, R.1; no longer IC1.PB5/PCINT5/!RESET!/ADC0/DW, R1.1, U$1.RST
- net VCC: now also BT1.+, C.1, IC2.VCC, J2.8, R.2; no longer C1.1, IC1.VCC, JP2.2, R1.2
Other:
- note added: "(c) 2019 Girolamo G"
- moved on the sheet: BT1, J1, U$1
